Commit message: Switching graphics to dae

File: src/main/resources/models/val_description/urdf/valkyrie_sim_arm_mass_sim.urdf (robot description, URDF)
Before this commit: robot valkyrie, 49 links, 48 joints
Links:
- link hokuyo_link: geometry 
- link leftAnklePitchLink: geometry visual mesh filename=package://val_description/model/meshes/legs/lj5.dae
- link leftElbowPitchLink: geometry visual mesh filename=package://val_description/model/meshes/arms/left_elbow_mass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
- link leftFoot: geometry visual mesh filename=package://val_description/model/meshes/legs/foot.dae
- link leftHipPitchLink: geometry visual mesh filename=package://val_description/model/meshes/legs/lj3_left.dae
- link leftHipYawLink: geometry visual mesh filename=package://val_description/model/meshes/legs/lj1_left.dae
- link leftKneePitchLink: geometry visual mesh filename=package://val_description/model/meshes/legs/lj4_left.dae
- link leftShoulderPitchLink: geometry visual mesh filename=package://val_description/model/meshes/arms/aj1_left.dae
- link leftShoulderRollLink: geometry visual mesh filename=package://val_description/model/meshes/arms/aj2_left.dae
- link leftShoulderYawLink: geometry visual mesh filename=package://val_description/model/meshes/arms/aj3_left.dae
- link lowerNeckPitchLink: geometry visual mesh filename=package://val_description/model/meshes/head/neckj1.dae
- link multisense/head: geometry 
- link neckYawLink: geometry visual mesh filename=package://val_description/model/meshes/head/neckj2.dae
- link pelvis: geometry visual mesh filename=package://val_description/model/meshes/pelvis/pelvis.dae
- link rightAnklePitchLink: geometry visual mesh filename=package://val_description/model/meshes/legs/lj5.dae
- link rightElbowPitchLink: geometry visual mesh filename=package://val_description/model/meshes/arms/right_elbow_mas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
- link rightFoot: geometry visual mesh filename=package://val_description/model/meshes/legs/foot.dae
- link rightHipPitchLink: geometry visual mesh filename=package://val_description/model/meshes/legs/lj3_right.dae
- link rightHipYawLink: geometry visual mesh filename=package://val_description/model/meshes/legs/lj1_right.dae
- link rightKneePitchLink: geometry visual mesh filename=package://val_description/model/meshes/legs/lj4_right.dae
- link rightShoulderPitchLink: geometry visual mesh filename=package://val_description/model/meshes/arms/aj1_right.dae
- link rightShoulderRollLink: geometry visual mesh filename=package://val_description/model/meshes/arms/aj2_right.dae
- link rightShoulderYawLink: geometry visual mesh filename=package://val_description/model/meshes/arms/aj3_right.dae
- link torso: geometry visual mesh filename=package://val_description/model/meshes/torso/torso.dae
- link torsoPitchLink: geometry visual mesh filename=package://val_description/model/meshes/torso/torsopitch.dae
- link torsoYawLink: geometry visual mesh filename=package://val_description/model/meshes/torso/torsoyaw.dae
- link upperNeckPitchLink: geometry visual mesh filename=package://val_description/model/meshes/head/head_multisense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

Commit message: update torso yaw limits

File: src/main/resources/models/val_description/urdf/valkyrie_sim_arm_mass_sim.urdf (robot description, URDF)
Before this commit: robot valkyrie, 49 links, 48 joints
Joints:
- joint torsoYaw: limit lower=-1.329 upper=1.181 effort=190 velocity=5.89 -> lower=-1.111 upper=1.111 effort=190 velocity=5.89

File: src/main/resources/models/val_description/urdf/valkyrie_sim_no_arms.urdf (robot description, URDF)
Before this commit: robot valkyrie, 41 links, 40 joints
Joints:
- joint torsoYaw: limit lower=-1.329 upper=1.181 effort=190 velocity=5.89 -> lower=-1.111 upper=1.111 effort=190 velocity=5.89

File: src/main/resources/models/val_description/urdf/valkyrie_sim_no_fingers.urdf (robot description, URDF)
Before this commit: robot valkyrie, 55 links, 54 joints
Joints:
- joint torsoYaw: limit lower=-1.329 upper=1.181 effort=190 velocity=5.89 -> lower=-1.111 upper=1.111 effort=190 velocity=5.89
